Commit message: update

File: ur_bringup/isaac/assets/ur16e_dualtool.urdf (robot description, URDF)
Before this commit: robot ur16e_dualtool, 12 links, 11 joints
Links:
- link gripper_2fg14__finger_left: mass 0.0567 -> 1.14685; geometry collision box size=0.07 0.074 0.082; visual box size=0.07 0.074 0.082
- link gripper_2fg14__finger_right: mass 0.0567 -> 1.14685; geometry collision box size=0.07 0.074 0.082; visual box size=0.07 0.074 0.082
Joints:
- joint gripper_2fg14__finger_left_joint: axis 0 1 0 -> 0 -1 0; origin xyz=0 0.013 0.08 rpy=0 0 0 -> xyz=0 0.03105 0.1144 rpy=0 0 0
- joint gripper_2fg14__finger_right_joint: axis 0 -1 0 -> 0 1 0; origin xyz=0 -0.013 0.08 rpy=0 0 0 -> xyz=0 -0.03105 0.1144 rpy=0 0 0

File: ur_bringup/urdf/ur16e_dualtool/ur16e_dualtool_eoat_macro.xacro (robot description, xacro)
@@ -80,18 +80,18 @@
     <link name="${prefix}gripper_2fg14__finger_left">
       <inertial>
-        <origin xyz="0 0 0.025" rpy="0 0 0"/>
-        <mass value="0.0567"/>
-        <inertia ixx="1.27386e-05" iyy="1.6065e-05" izz="5.1786e-06" ixy="0" ixz="0" iyz="0"/>
-      </inertial>
-      <collision>
-        <origin xyz="0 0 0.025" rpy="0 0 0"/>
-        <geometry>
-          <box size="0.03 0.014 0.05"/>
-        </geometry>
-      </collision>
-      <visual>
-        <origin xyz="0 0 0.025" rpy="0 0 0"/>
-        <geometry>
-          <box size="0.03 0.014 0.05"/>
+        <origin xyz="0 0 0.041" rpy="0 0 0"/>
+        <mass value="1.14685"/>
+        <inertia ixx="0.00116597" iyy="0.00111092" izz="0.000991645" ixy="0" ixz="0" iyz="0"/>
+      </inertial>
+      <collision>
+        <origin xyz="0 0 0" rpy="0 0 0"/>
+        <geometry>
+          <mesh filename="package://ur_bringup/meshes/eoat/gripper_2fg14__finger_left_col.obj"/>
+        </geometry>
+      </collision>
+      <visual>
+        <origin xyz="0 0 0" rpy="0 0 0"/>
+        <geometry>
+          <mesh filename="package://ur_bringup/meshes/eoat/gripper_2fg14__finger_left.obj"/>
         </geometry>
       </visual>
@@ -99,18 +99,18 @@
     <link name="${prefix}gripper_2fg14__finger_right">
       <inertial>
-        <origin xyz="0 0 0.025" rpy="0 0 0"/>
-        <mass value="0.0567"/>
-        <inertia ixx="1.27386e-05" iyy="1.6065e-05" izz="5.1786e-06" ixy="0" ixz="0" iyz="0"/>
-      </inertial>
-      <collision>
-        <origin xyz="0 0 0.025" rpy="0 0 0"/>
-        <geometry>
-          <box size="0.03 0.014 0.05"/>
-        </geometry>
-      </collision>
-      <visual>
-        <origin xyz="0 0 0.025" rpy="0 0 0"/>
-        <geometry>
-          <box size="0.03 0.014 0.05"/>
+        <origin xyz="0 0 0.041" rpy="0 0 0"/>
+        <mass value="1.14685"/>
+        <inertia ixx="0.00116597" iyy="0.00111092" izz="0.000991645" ixy="0" ixz="0" iyz="0"/>
+      </inertial>
+      <collision>
+        <origin xyz="0 0 0" rpy="0 0 0"/>
+        <geometry>
+          <mesh filename="package://ur_bringup/meshes/eoat/gripper_2fg14__finger_right_col.obj"/>
+        </geometry>
+      </collision>
+      <visual>
+        <origin xyz="0 0 0" rpy="0 0 0"/>
+        <geometry>
+          <mesh filename="package://ur_bringup/meshes/eoat/gripper_2fg14__finger_right.obj"/>
         </geometry>
       </visual>
@@ -234,6 +234,6 @@
       <parent link="${prefix}gripper_2fg14"/>
       <child link="${prefix}gripper_2fg14__finger_left"/>
-      <origin xyz="0 0.013 0.08" rpy="0 0 0"/>
-      <axis xyz="0 1 0"/>
+      <origin xyz="0 0.03105 0.1144" rpy="0 0 0"/>
+      <axis xyz="0 -1 0"/>
       <limit lower="0" upper="0.025" effort="140" velocity="0.45"/>
       <dynamics damping="0" friction="0"/>
@@ -242,6 +242,6 @@
       <parent link="${prefix}gripper_2fg14"/>
       <child link="${prefix}gripper_2fg14__finger_right"/>
-      <origin xyz="0 -0.013 0.08" rpy="0 0 0"/>
-      <axis xyz="0 -1 0"/>
+      <origin xyz="0 -0.03105 0.1144" rpy="0 0 0"/>
+      <axis xyz="0 1 0"/>
       <limit lower="0" upper="0.025" effort="140" velocity="0.45"/>
       <dynamics damping="0" friction="0"/>
